File: KITTY_MKII/Ignition_Module.kicad_pcb (KiCad board)
At the start: 2 copper layers, 82 x 55 mm, 57 parts, among them J1 Conn_01x01_Pin, J10 Conn_01x01_Pin, J11 Conn_01x01_Pin, J12 Conn_01x01_Pin, J13 Conn_01x01_Pin, J14 Conn_01x01_Pin, J15 Conn_01x01_Pin, J16 Conn_01x01_Pin, J2 Conn_01x01_Pin, J3 Conn_01x01_Pin, J4 Conn_01x01_Pin, J5 Conn_01x01_Pin, J6 Conn_01x01_Pin, J7 Conn_01x01_Pin, J8 Conn_01x01_Pin, J9 Conn_01x01_Pin, Q1 Q_NIGBT_ECG, Q2 Q_NIGBT_ECG, Q3 Q_NIGBT_ECG, Q4 Q_NIGBT_ECG

Commit message: working on enclosure
Parts:
- added HS1: Heatsink, Heatsink:Heatsink_Fischer_FK24413DPAK_23x13mm, B.Cu at (170.2, 83.4)
- added HS1: Heatsink, Heatsink:Heatsink_Fischer_FK24413DPAK_23x13mm, B.Cu at (118.3, 83.4)
- added HS1: Heatsink, Heatsink:Heatsink_Fischer_FK24413DPAK_23x13mm, B.Cu at (170.2, 68.6)
- added HS1: Heatsink, Heatsink:Heatsink_Fischer_FK24413DPAK_23x13mm, B.Cu at (118.3, 68.8)
- renumbered D3 to D1, D5 to D3, D1 to D5, D2 to D6, J11 to J1, J6 to J10, J8 to J11, J15 to J12, J7 to J13, J5 to J14, J3 to J15, J1 to J16, J14 to J2, J9 to J3, J10 to J4, J12 to J5, J13 to J6, J16 to J7, J2 to J8, J4 to J9, R5 to R1, R7 to R3, R8 to R4, R3 to R5, R4 to R6, R1 to R9, TP5 to TP3, TP6 to TP4, TP3 to TP5, TP4 to TP6
Connections:
- D1 pad 1: Net-(D1-A) -> Net-(D1-K)
- D3 pad 1: Net-(D7-K) -> /Net-(D7-K)
- D5 pad 2: Net-(D1-A) -> Net-(D1-K)
- D6 pad 2: Net-(D3-K) -> /Net-(D3-K)
- D7 pad 1: Net-(D8-K) -> /Net-(D8-K)
- D7 pad 2: Net-(D7-K) -> /Net-(D7-K)
- D8 pad 1: Net-(D11-K) -> /Net-(D11-K)
- D8 pad 2: Net-(D10-K) -> Net-(D4-K)
- R1 pad 2: Net-(D1-A) -> Net-(D1-K)
- R11 pad 1: Net-(D7-K) -> /Net-(D7-K)
- R12 pad 1: Net-(D10-K) -> Net-(D4-K)
- R3 pad 2: Net-(D7-K) -> /Net-(D7-K)
- R4 pad 2: Net-(D10-K) -> Net-(D4-K)
- R9 pad 1: Net-(D1-A) -> Net-(D1-K)
