File: KITTY_MKII/Ignition_Module.kicad_sch (KiCad schematic)
At the start: 49 parts, among them J1 Conn_01x01_Pin, J10 Conn_01x01_Pin, J11 Conn_01x01_Pin, J12 Conn_01x01_Pin, J13 Conn_01x01_Pin, J14 Conn_01x01_Pin, J15 Conn_01x01_Pin, J16 Conn_01x01_Pin, J2 Conn_01x01_Pin, J3 Conn_01x01_Pin, J4 Conn_01x01_Pin, J5 Conn_01x01_Pin, J6 Conn_01x01_Pin, J7 Conn_01x01_Pin, J8 Conn_01x01_Pin, J9 Conn_01x01_Pin, Q5 Q_NIGBT_ECG, Q6 Q_NIGBT_ECG, Q7 Q_NIGBT_ECG, Q8 Q_NIGBT_ECG

Commit message: working on enclosure
Parts:
- added HS1, HS2, HS3, HS4: Heatsink, Heatsink:Heatsink_Fischer_FK24413DPAK_23x13mm, symbol Mechanical:Heatsink
- renumbered C7 to C3, D3 to D1, D3 to D2, D5 to D3, D10 to D4, D1 to D5, D2 to D6, J11 to J1, J6 to J10, J8 to J11, J15 to J12, J7 to J13, J5 to J14, J3 to J15, J1 to J16, J14 to J2, J9 to J3, J10 to J4, J12 to J5, J13 to J6, J16 to J7, J2 to J8, J4 to J9, Q5 to Q1, Q6 to Q2, Q7 to Q3, Q8 to Q4, R5 to R1, R8 to R10, R5 to R2, R7 to R3, R8 to R4, R3 to R5, R4 to R6, R12 to R7, R17 to R8, R1 to R9, TP5 to TP3, TP6 to TP4, TP3 to TP5, TP4 to TP6
Connections:
- net Net-(D3-K): now reaches D2.1 (K), D6.2 (A), Q2.1 (G), R10.1, R2.2
- net Net-(D11-K): now reaches D8.1 (K), R8.1
- net Net-(D7-K): now reaches D3.1 (K), D7.2 (A), Q3.1 (G), R11.1, R3.2
- net Net-(D8-K): now reaches D7.1 (K), R7.1
- net Net-(D5-K): now reaches D6.1 (K), R6.1
